File: Connectors.kicad_sch (KiCad schematic)
At the start: 16 parts, among them CN901 XT60PW-M, CN902 1053131202, CN903 1053131202, CN904 1053131203, CN905 1053131203, CN906 1053131204, CN907 1053131204, CN908 1053131204, J901 USB_C_Receptacle_USB2.0

Commit message: dont like direction, doing too much
Parts:
- renumbered CN905 to CN904, CN904 to CN905, D903 to D902, D902 to D903, D905 to D904, D904 to D905
