File: FPGA.kicad_sch (KiCad schematic)
At the start: 40 parts, among them J401 Conn_01x06_Pin, U401 LFE5U-45F-6TG144C

Commit message: dont like direction, doing too much
Parts:
- renumbered C416 to C414, C414 to C415, C415 to C416, C427 to C419, C419 to C420, C420 to C421, C421 to C422, C422 to C423, C423 to C424, C424 to C425, C425 to C426, C426 to C427, C430 to C429, C432 to C430, C434 to C431, C436 to C432
Connections:
- net FLASH_SPI_CS renamed FPGA_FLASH_SPI.CS
- net FLASH_SPI_MISO renamed FPGA_FLASH_SPI.MISO
- net FLASH_SPI_MOSI renamed FPGA_FLASH_SPI.MOSI
- net FLASH_SPI_SCK renamed FPGA_FLASH_SPI.SCK
