File: Flash.kicad_sch (KiCad schematic)
At the start: 3 parts, among them U802 MX25L3233FZBI-08QTR

Commit message: dont like direction, doing too much
Parts:
- renumbered R802 to R801, U802 to U801
Connections:
- net FPGA_CS renamed FLASH_SPI.CS
- net FPGA_MISO renamed FLASH_SPI.MISO
- net FPGA_MOSI renamed FLASH_SPI.MOSI
- net FPGA_SCK renamed FLASH_SPI.SCK
Other:
- note added: "need to check this is even possible, two devices talking to one flash chip. non-trivial"
