File: GNSS.kicad_pcb (KiCad board)
At the start: 4 copper layers, 100 x 50 mm, 225 parts, among them CN901 XT60PW-M, CN902 1053131202, CN903 1053131202, CN904 1053131203, CN905 1053131203, CN906 1053131204, CN907 1053131204, CN908 1053131204, IC301 STM32H743ZIT6TR, IC601 IIM-20670, IC602 DPS368XTSA1, IC603 ICM-42688-P, IC604 BMP390, J101 Conn_Coaxial, J102 Conn_Coaxial, J401 Conn_01x06_Pin, J901 USB_C_Receptacle_USB2.0, Q201 IRF7324, Q202 IRF7324, SW301 SW_Push, SW302 SW_Push, U201 LTC4417IGN, U202 TPS566238RQFR, U203 TLV75525PDRV, U204 TPS566238RQFR, U205 TPS55289RYQR, U301 ABM8G-25.000MHZ-B4Y-T, U401 LFE5U-45F-6TG144C, U501 MAX2769BETI/V+, U701 RM3100, U802 MX25L3233FZBI-08QTR, Y101 TG2016SMN 16.3680M-MCGNNMB

Commit message: dont like direction, doing too much
Parts:
- added R305: 10kΩ, Resistor_SMD:R_0402_1005Metric, B.Cu at (106.5, 65.1)
- added R306: 10kΩ, Resistor_SMD:R_0402_1005Metric, F.Cu at (77.8, 79.2)
- C201, C202, R206, R207, R208, U201: moved to B.Cu
- R211: renamed from R209; moved to B.Cu
- R212: renamed from R210; moved to B.Cu
- R213: renamed from R211; moved to B.Cu
- R214: renamed from R212; moved to B.Cu
- moved SW302 65.1 mm to (134.2, 40.4)
- moved C301 62.8 mm to (134.6, 38.0)
- moved R301 60.6 mm to (134.4, 36.8)
- moved R302 59.4 mm to (126.9, 37.0)
- moved SW301 56.9 mm to (129.0, 39.9)
- moved R304 55.2 mm to (69.3, 59.8), turned to 0 degrees
- moved R303 54.1 mm to (69.3, 57.8), turned to 0 degrees
- moved C210 9.21 mm to (101.3, 83.5), turned to -90 degrees
- moved C208 8.86 mm to (95.8, 83.5), turned to 90 degrees
- moved Q201 8.70 mm to (96.4, 78.9)
- moved Q202 8.70 mm to (101.9, 78.9)
- moved R214 6.28 mm to (102.6, 83.4)
- moved R211 4.28 mm to (101.6, 84.8)
- moved C202 3.28 mm to (101.1, 86.5), turned to 0 degrees
- moved R212 3.28 mm to (101.1, 83.4), turned to 0 degrees
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- renumbered C235 to C203, C236 to C204, C204 to C205, C205 to C207, C207 to C209, C209 to C211, C215 to C214, C211 to C215, C234 to C216, C216 to C217, C214 to C218, C203 to C219, C221 to C220, C220 to C221, C218 to C222, C217 to C223, C223 to C224, C224 to C225, C225 to C226, C226 to C227, C227 to C228, C228 to C229, C229 to C230, C232 to C231, C231 to C232, C230 to C234, C304 to C302, C305 to C303, C307 to C304, C302 to C305, C303 to C307, C416 to C414, C414 to C415, C415 to C416, C427 to C419, C419 to C420, C420 to C421, C421 to C422, C422 to C423, C423 to C424, C424 to C425, C425 to C426, C426 to C427, C430 to C429, C432 to C430, C434 to C431, C436 to C432, C502 to C501, C504 to C502, C501 to C503, C503 to C504, CN905 to CN904, CN904 to CN905, D903 to D902, D902 to D903, D905 to D904, D904 to D905, R220 to R209, R221 to R210, R223 to R215, R222 to R216, R213 to R217, R214 to R218, R215 to R219, R216 to R220, R217 to R221, R218 to R222, R219 to R223, R302 to R301, R301 to R302, R802 to R801, SW302 to SW301, SW301 to SW302, U802 to U801
Connections:
- net /Flash/CS renamed /FPGA/FPGA_FLASH_SPI.CS
- net /Flash/MISO renamed /FPGA/FPGA_FLASH_SPI.MISO
- net /Flash/MOSI renamed /FPGA/FPGA_FLASH_SPI.MOSI
- net /Flash/SCK renamed /FPGA/FPGA_FLASH_SPI.SCK
- IC301 pad 10: /MCU/SDA_PWR -> /Connectors/SDA_0
- IC301 pad 11: /MCU/SCL_PWR -> /Connectors/SCL_0
- IC301 pad 134: unconnected-(IC301-PB4-Pad134) -> /Connectors/UART_TX
- IC301 pad 135: unconnected-(IC301-PB5-Pad135) -> /Connectors/UART_RX
- IC301 pad 26: unconnected-(IC301-PC0-Pad26) -> +1V1
- IC301 pad 27: unconnected-(IC301-PC1-Pad27) -> /MCU/1v1_enable
- IC301 pad 28: unconnected-(IC301-PC2_C-Pad28) -> +2V5
- IC301 pad 29: unconnected-(IC301-PC3_C-Pad29) -> /MCU/2v5_enable
- IC301 pad 41: unconnected-(IC301-PA5-Pad41) -> /MCU/SERVO_PWR_FAULT
- IC301 pad 42: unconnected-(IC301-PA6-Pad42) -> /MCU/Batt_Volt_Monitor
- IC301 pad 54: /MCU/Batt_Volt_Monitor -> /MCU/SCL_PWR
- IC301 pad 55: unconnected-(IC301-PF15-Pad55) -> /MCU/SDA_PWR
- R303 pad 1: /MCU/SCL_PWR -> +1V1
- R303 pad 2: +3V3 -> GND
- R304 pad 1: /MCU/SDA_PWR -> +2V5
- R304 pad 2: +3V3 -> GND
Routing:
- net /MCU/BOOT: track 53.9 -> 4.97 mm
- net /MCU/NRST: track 47.0 -> 1.30 mm
- net /MCU/SDA_PWR: track 36.5 -> 13.3 mm
- net /MCU/SCL_PWR: track 35.2 -> 13.6 mm
- net /Power/BATT: track 45.4 -> 29.9 mm, vias 0 -> 1
- net Net-(U201-VOUT): track 14.6 -> 7.51 mm, vias 2 -> 1
- net Net-(Q201A-S1): track 7.62 -> 13.2 mm, vias 0 -> 1
- net /Connectors/VBUS: track 80.3 -> 75.8 mm, vias 3 -> 5
- net /MCU/Batt_Volt_Monitor: track 3.75 -> 0.95 mm
- net Net-(Q201A-G1): track 8.61 -> 11.0 mm, vias 0 -> 1
- net +3V3: track 121.6 -> 119.4 mm, vias 56 -> 54
- net Net-(Q202A-G1): track 7.97 -> 9.91 mm, vias 0 -> 1
- net Net-(Q202A-S1): track 10.1 -> 10.4 mm, vias 0 -> 1
- net GND: vias 192 -> 178
