File: GNSS.kicad_sch (KiCad schematic)
At the start: 8 parts, among them J101 Conn_Coaxial, J102 Conn_Coaxial, Y101 TG2016SMN 16.3680M-MCGNNMB

Commit message: dont like direction, doing too much
Other:
- sheet FPGA ports: added FPGA_FLASH_SPI{SCK MOSI MISO CS}; removed FLASH_SPI_CS, FLASH_SPI_MISO, FLASH_SPI_MOSI, FLASH_SPI_SCK
- sheet Flash ports: added FLASH_SPI{SCK MOSI MISO CS}; removed FPGA_CS, FPGA_MISO, FPGA_MOSI, FPGA_SCK, MCU_CS, MCU_MISO, MCU_MOSI, MCU_SCK
- sheet MCU ports: added MCU_FLASH_SPI{SCK MOSI MISO CS}; removed none
