File: MCU.kicad_sch (KiCad schematic)
At the start: 30 parts, among them IC301 STM32H743ZIT6TR, SW301 SW_Push, SW302 SW_Push, U301 ABM8G-25.000MHZ-B4Y-T

Commit message: dont like direction, doing too much
Parts:
- added R305, R306: 10kΩ, Resistor_SMD:R_0402_1005Metric, symbol Device:R_Small
- renumbered C304 to C302, C305 to C303, C307 to C304, C302 to C305, C303 to C307, R302 to R301, R301 to R302, SW302 to SW301, SW301 to SW302
Connections:
- net +3V3: now also R305.2, R306.2; no longer R303.2, R304.2
- net 1v1_enable: now also IC301.27 (PC1)
- net 2v5_enable: now also IC301.29 (PC3_C)
- net Batt_Volt_Monitor: now also IC301.42 (PA6); no longer IC301.54 (PF14)
- net GND: now also R303.2, R304.2
- net SCL: now also IC301.11 (PF1)
- net SCL_PWR: now also IC301.54 (PF14), R305.1; no longer IC301.11 (PF1), R303.1
- net SDA: now also IC301.10 (PF0)
- net SDA_PWR: now also IC301.55 (PF15), R306.1; no longer IC301.10 (PF0), R304.1
- net SERVO_PWR_FAULT: now also IC301.41 (PA5)
- net UART_RX: now also IC301.135 (PB5)
- net UART_TX: now also IC301.134 (PB4)
- net +1V1: now reaches IC301.26 (PC0)
- net +1V1: now also R303.1
- net +2V5: now reaches IC301.28 (PC2_C)
- net +2V5: now also R304.1
Other:
- moved on the sheet: C305, C307, U301
