File: Power.kicad_sch (KiCad schematic)
At the start: 72 parts, among them Q201 IRF7324, Q202 IRF7324, U201 LTC4417IGN, U202 TPS566238RQFR, U203 TLV75525PDRV, U204 TPS566238RQFR, U205 TPS55289RYQR

Commit message: dont like direction, doing too much
Parts:
- C230: renamed from C229; value ~ -> (none)
- renumbered C235 to C203, C236 to C204, C204 to C205, C205 to C207, C207 to C209, C209 to C211, C215 to C214, C211 to C215, C234 to C216, C216 to C217, C214 to C218, C203 to C219, C221 to C220, C220 to C221, C218 to C222, C217 to C223, C223 to C224, C224 to C225, C225 to C226, C226 to C227, C227 to C228, C228 to C229, C232 to C231, C231 to C232, C230 to C234, R220 to R209, R221 to R210, R209 to R211, R210 to R212, R211 to R213, R212 to R214, R223 to R215, R222 to R216, R213 to R217, R214 to R218, R215 to R219, R216 to R220, R217 to R221, R218 to R222, R219 to R223
