File: RF_Frontend.kicad_sch (KiCad schematic)
At the start: 26 parts, among them U501 MAX2769BETI/V+

Commit message: dont like direction, doing too much
Parts:
- renumbered C502 to C501, C504 to C502, C501 to C503, C503 to C504
